File: template/d1_mini_shield.kicad_pcb (KiCad board)
At the start: 2 copper layers, 25.7 x 34.4 mm, 3 parts, among them P1 CONN_01X08, P2 CONN_01X08

Commit message: Updated template & library to KiCad 8 format
All legacy files have been converted to the corresponding
current KiCad 8.x file formats, unnecessary files have
been removed. The original pin header symbols `CONN_01X08`
have been mapped to the symbol `Connector_Generic:Conn_01x08`
that is included with KiCad.

The README was updated with current instructions.
Other:
- net class Default removed
